File: pcb/bike lights.kicad_sch (KiCad schematic)
At the start: 42 parts, among them SW1 Power, SW2 SW_SPDT_MSM, U1 MSP430G2533IN20, U2 74AHC595, U3 74AHC595

Commit message: Update schematics
Connections:
- net at U1.4 (TA0.1/UCA0TXD/UCA0SIMO/A2/P1.2): now also U2.11 (SRCLK), U3.11 (SRCLK); no longer U2.12 (RCLK)
- net at U2.14 (SER), U3.14 (SER): now also U1.5 (ADC10CLK/VREF-/VeREF-/A3/P1.3); no longer U1.6 (TCK/SMCLK/UCB0STE/UCA0CLK/VREF+/VeREF+/A4/P1.4)
- new net: U1.6 (TCK/SMCLK/UCB0STE/UCA0CLK/VREF+/VeREF+/A4/P1.4), U2.12 (RCLK)
Other:
- note added: "CLOCK"
- note added: "DATA"
- note added: "LATCH_A"
- note added: "LATCH_B"
Changed lines of the file:
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@@
   (junction (at 46.99 149.86) (diameter 0) (color 0 0 0 0)
   )
+  (junction (at 153.67 85.09) (diameter 0) (color 0 0 0 0)
+  )
   (junction (at 264.16 64.77) (diameter 0) (color 0 0 0 0)
   )
   (junction (at 264.16 69.85) (diameter 0) (color 0 0 0 0)
   )
+  (junction (at 147.32 82.55) (diameter 0) (color 0 0 0 0)
+  )
   (junction (at 264.16 59.69) (diameter 0) (color 0 0 0 0)
   )
@@
   (junction (at 264.16 54.61) (diameter 0) (color 0 0 0 0)
   )
-  (junction (at 147.32 85.09) (diameter 0) (color 0 0 0 0)
-  )
   (junction (at 264.16 80.01) (diameter 0) (color 0 0 0 0)
   )
-  (junction (at 153.67 87.63) (diameter 0) (color 0 0 0 0)
-  )
   (junction (at 264.16 133.35) (diameter 0) (color 0 0 0 0)
   )
@@
     (stroke (width 0) (type default))
   )
+  (wire (pts (xy 153.67 85.09) (xy 153.67 138.43))
+    (stroke (width 0) (type default))
+  )
   (wire (pts (xy 250.19 148.59) (xy 264.16 148.59))
     (stroke (width 0) (type default))
@@
     (stroke (width 0) (type default))
   )
-  (wire (pts (xy 147.32 69.85) (xy 147.32 85.09))
-    (stroke (width 0) (type default))
-  )
-  (wire (pts (xy 123.19 87.63) (xy 153.67 87.63))
-    (stroke (width 0) (type default))
-  )
   (wire (pts (xy 35.56 53.34) (xy 58.42 53.34))
     (stroke (width 0) (type default))
@@
     (stroke (width 0) (type default))
   )
-  (wire (pts (xy 123.19 85.09) (xy 147.32 85.09))
-    (stroke (width 0) (type default))
-  )
   (wire (pts (xy 250.19 80.01) (xy 264.16 80.01))
     (stroke (width 0) (type default))
@@
     (stroke (width 0) (type default))
   )
-  (wire (pts (xy 123.19 82.55) (xy 140.97 82.55))
-    (stroke (width 0) (type default))
-  )
   (wire (pts (xy 166.37 123.19) (xy 176.53 123.19))
     (stroke (width 0) (type default))
@@
     (stroke (width 0) (type default))
   )
-  (wire (pts (xy 153.67 74.93) (xy 153.67 87.63))
-    (stroke (width 0) (type default))
-  )
   (wire (pts (xy 140.97 90.17) (xy 140.97 125.73))
     (stroke (width 0) (type default))
@@
     (stroke (width 0) (type default))
   )
+  (wire (pts (xy 123.19 85.09) (xy 153.67 85.09))
+    (stroke (width 0) (type default))
+  )
   (wire (pts (xy 226.06 54.61) (xy 210.82 54.61))
     (stroke (width 0) (type default))
@@
     (stroke (width 0) (type default))
   )
+  (wire (pts (xy 123.19 87.63) (xy 140.97 87.63))
+    (stroke (width 0) (type default))
+  )
   (wire (pts (xy 250.19 64.77) (xy 264.16 64.77))
     (stroke (width 0) (type default))
@@
     (stroke (width 0) (type default))
   )
-  (wire (pts (xy 153.67 87.63) (xy 153.67 138.43))
+  (wire (pts (xy 153.67 74.93) (xy 153.67 85.09))
+    (stroke (width 0) (type default))
+  )
+  (wire (pts (xy 123.19 82.55) (xy 147.32 82.55))
     (stroke (width 0) (type default))
   )
@@
     (stroke (width 0) (type default))
   )
-  (wire (pts (xy 147.32 85.09) (xy 147.32 133.35))
+  (wire (pts (xy 147.32 69.85) (xy 147.32 82.55))
     (stroke (width 0) (type default))
   )
@@
     (stroke (width 0) (type default))
   )
-  (wire (pts (xy 140.97 82.55) (xy 140.97 62.23))
+  (wire (pts (xy 140.97 62.23) (xy 140.97 87.63))
     (stroke (width 0) (type default))
   )
@@
     (stroke (width 0) (type default))
   )
+  (wire (pts (xy 147.32 82.55) (xy 147.32 133.35))
+    (stroke (width 0) (type default))
+  )
   (wire (pts (xy 250.19 74.93) (xy 264.16 74.93))
     (stroke (width 0) (type default))
@@
     (stroke (width 0) (type default))
   )
+  (text "DATA" (at 127 85.09 0)
+    (effects (font (size 1 1) (color 132 132 132 1)) (justify left bottom))
+  )
+  (text "LATCH_A" (at 127 87.63 0)
+    (effects (font (size 1 1) (color 132 132 132 1)) (justify left bottom))
+  )
+  (text "LATCH_B" (at 127 90.17 0)
+    (effects (font (size 1 1) (color 132 132 132 1)) (justify left bottom))
+  )
+  (text "CLOCK" (at 127 82.55 0)
+    (effects (font (size 1 1) (color 132 132 132 1)) (justify left bottom))
+  )
   (symbol (lib_id "MCU_Texas_MSP430:MSP430G2533IN20") (at 85.09 87.63 0) (unit 1)
